Commit message: updates

File: vega_description/urdf/vega_description.xacro (robot description, xacro)
@@ -36,5 +36,5 @@
       <origin
         xyz="0 0 0"
-        rpy="0 0 0" />
+        rpy="1.571 0 0" />
       <geometry>
         <mesh
@@ -499,5 +499,5 @@
     <collision>
       <origin
-        xyz="0 0 0"
+        xyz="0.075 -0.05 0"
         rpy="0 0 0" />
       <geometry>
@@ -575,3 +575,68 @@
       xyz="0 1 0" />
   </joint>
+  <link
+    name="Link_11">
+    <inertial>
+      <origin
+        xyz="0.151523838773093 0.0120793005495848 -0.00451680024396695"
+        rpy="0 0 0" />
+      <mass
+        value="0.0676472542576388" />
+      <inertia
+        ixx="3.54922400123965E-06"
+        ixy="-2.99865301015401E-16"
+        ixz="4.85967691354056E-15"
+        iyy="0.000543285324126437"
+        iyz="1.19005104729777E-08"
+        izz="0.000541662726314469" />
+    </inertial>
+  </link>
+  <joint
+    name="Joint_5_11"
+    type="fixed">
+    <origin
+      xyz="0.030 -0.020 0"
+      rpy="0 0 0" />
+    <parent
+      link="Link_5" />
+    <child
+      link="Link_11" />
+    <axis
+      xyz="0 1 0" />
+  </joint>
+  <link
+    name="Link_Tool">
+    <inertial>
+      <origin
+        xyz="0.151523838773093 0.0120793005495848 -0.00451680024396695"
+        rpy="0 0 0" />
+      <mass
+        value="0.0676472542576388" />
+      <inertia
+        ixx="3.54922400123965E-06"
+        ixy="-2.99865301015401E-16"
+        ixz="4.85967691354056E-15"
+        iyy="0.000543285324126437"
+        iyz="1.19005104729777E-08"
+        izz="0.000541662726314469" />
+    </inertial>
+  </link>
+  <joint
+    name="Joint_11_Tool"
+    type="revolute">
+    <origin
+      xyz="0.030 0 0"
+      rpy="0 0 0" />
+    <parent
+      link="Link_11" />
+    <child
+      link="Link_Tool" />
+    <axis
+      xyz="0 1 0" />
+    <limit
+      lower="-3.142"
+      upper="3.142"
+      effort="10"
+      velocity="2.094" />
+  </joint>
 </robot>

File: vega_description/urdf/vega_description_chain.xacro (robot description, xacro)
@@ -1,4 +1,5 @@
 <?xml version="1.0" encoding="utf-8"?>
 <robot
+  xmlns:xacro="http://www.ros.org/wiki/xacro"
   name="vega_description">
   <link
@@ -35,5 +36,5 @@
       <origin
         xyz="0 0 0"
-        rpy="0 0 0" />
+        rpy="1.571 0 0" />
       <geometry>
         <mesh
@@ -200,5 +201,5 @@
   <joint
     name="Joint_3_4"
-    type="continuous">
+    type="revolute">
     <origin
       xyz="0.25 0.055 0"
@@ -210,4 +211,9 @@
     <axis
       xyz="0 -1 0" />
+    <limit
+      lower="-3.142"
+      upper="3.142"
+      effort="15"
+      velocity="2.094" />
   </joint>
   <link
@@ -253,5 +259,5 @@
   <joint
     name="Joint_4_5"
-    type="continuous">
+    type="revolute">
     <origin
       xyz="0.3 0.025 0"
@@ -263,4 +269,9 @@
     <axis
       xyz="0 0 1" />
+    <limit
+      lower="-3.142"
+      upper="3.142"
+      effort="10"
+      velocity="2.094" />
   </joint>
   <link
@@ -304,7 +315,11 @@
     </collision>
   </link>
-  <joint
-    name="Joint_2_6"
-    type="revolute">
+  <link
+    name="Link_2_6">
+  </link>
+    <joint
+    name="Joint_2_6_1"
+    type="continuous">
+    <mimic joint="Joint_2_3" multiplier="-1" offset="0"/>
     <origin
       xyz="0.02 0.085 -0.0285"
@@ -313,12 +328,21 @@
       link="Link_2" />
     <child
+      link="Link_2_6" />
+    <axis
+      xyz="0 0 1" />
+  </joint>
+  <joint
+    name="Joint_2_6_2"
+    type="continuous">
+    <mimic joint="Joint_3_4" multiplier="-1" offset="0"/>
+    <origin
+      xyz="0 0 0"
+      rpy="0 0 0" />
+    <parent
+      link="Link_2_6" />
+    <child
       link="Link_6" />
     <axis
       xyz="0 0 1" />
-    <limit
-      lower="-3.142"
-      upper="3.142"
-      effort="15"
-      velocity="2.094" />
   </joint>
   <link
@@ -365,4 +389,5 @@
     name="Joint_6_7"
     type="continuous">
+    <mimic joint="Joint_3_4" multiplier="1" offset="0"/>
     <origin
       xyz="-0.115 0 0.025"
@@ -418,4 +443,5 @@
     name="Joint_2_8"
     type="continuous">
+    <mimic joint="Joint_2_3" multiplier="-1" offset="0"/>
     <origin
       xyz="-0.055 0.135 0.049"
@@ -460,5 +486,5 @@
     <collision>
       <origin
-        xyz="0 0 0"
+        xyz="0.075 -0.05 0"
         rpy="0 0 0" />
       <geometry>
@@ -471,4 +497,5 @@
     name="Joint_8_9"
     type="continuous">
+    <mimic joint="Joint_2_3" multiplier="1" offset="0"/>
     <origin
       xyz="0.25 -0.0175 0"
@@ -521,7 +548,11 @@
     </collision>
   </link>
-  <joint
-    name="Joint_9_10"
+  <link
+    name="Link_9_10">
+  </link>
+  <joint
+    name="Joint_9_10_1"
     type="continuous">
+    <mimic joint="Joint_2_3" multiplier="-1" offset="0"/>
     <origin
       xyz="0.095 -0.015 0.0175"
@@ -530,7 +561,86 @@
       link="Link_9" />
     <child
+      link="Link_9_10" />
+    <axis
+      xyz="0 1 0" />
+  </joint>
+  <joint
+    name="Joint_9_10_2"
+    type="continuous">
+    <mimic joint="Joint_3_4" multiplier="-1" offset="0"/>
+    <origin
+      xyz="0 0 0"
+      rpy="0 0 0" />
+    <parent
+      link="Link_9_10" />
+    <child
       link="Link_10" />
     <axis
       xyz="0 1 0" />
   </joint>
+  <link
+    name="Link_11">
+    <inertial>
+      <origin
+        xyz="0.151523838773093 0.0120793005495848 -0.00451680024396695"
+        rpy="0 0 0" />
+      <mass
+        value="0.0676472542576388" />
+      <inertia
+        ixx="3.54922400123965E-06"
+        ixy="-2.99865301015401E-16"
+        ixz="4.85967691354056E-15"
+        iyy="0.000543285324126437"
+        iyz="1.19005104729777E-08"
+        izz="0.000541662726314469" />
+    </inertial>
+  </link>
+  <joint
+    name="Joint_5_11"
+    type="fixed">
+    <origin
+      xyz="0.030 -0.020 0"
+      rpy="0 0 0" />
+    <parent
+      link="Link_5" />
+    <child
+      link="Link_11" />
+    <axis
+      xyz="0 1 0" />
+  </joint>
+  <link
+    name="Link_Tool">
+    <inertial>
+      <origin
+        xyz="0.151523838773093 0.0120793005495848 -0.00451680024396695"
+        rpy="0 0 0" />
+      <mass
+        value="0.0676472542576388" />
+      <inertia
+        ixx="3.54922400123965E-06"
+        ixy="-2.99865301015401E-16"
+        ixz="4.85967691354056E-15"
+        iyy="0.000543285324126437"
+        iyz="1.19005104729777E-08"
+        izz="0.000541662726314469" />
+    </inertial>
+  </link>
+  <joint
+    name="Joint_11_Tool"
+    type="revolute">
+    <origin
+      xyz="0.030 0 0"
+      rpy="0 0 0" />
+    <parent
+      link="Link_11" />
+    <child
+      link="Link_Tool" />
+    <axis
+      xyz="0 1 0" />
+    <limit
+      lower="-3.142"
+      upper="3.142"
+      effort="10"
+      velocity="2.094" />
+  </joint>
 </robot>

Commit message: updated meshes

File: vega_description/urdf/vega_description.xacro (robot description, xacro)
@@ -25,5 +25,5 @@
       <geometry>
         <mesh
-          filename="package://vega_description/meshes/Link_1.STL" />
+          filename="package://vega_description/meshes/Link_1.STL"/>
       </geometry>
       <material
@@ -252,19 +252,21 @@
       <geometry>
         <mesh
-          filename="package://vega_description/meshes/Link_5.STL" />
-      </geometry>
-      <material
-        name="">
-        <color
-          rgba="0.752941176470588 0.752941176470588 0.752941176470588 1" />
-      </material>
-    </visual>
-    <collision>
-      <origin
-        xyz="0 0 0"
-        rpy="0 0 0" />
-      <geometry>
-        <mesh
-          filename="package://vega_description/meshes/Link_5.STL" />
+          filename="package://vega_description/meshes/Link_5.STL"
+          scale="0.001 0.001 0.001" />
+      </geometry>
+      <material
+        name="">
+        <color
+          rgba="0.752941176470588 0.752941176470588 0.752941176470588 1" />
+      </material>
+    </visual>
+    <collision>
+      <origin
+        xyz="0 0 0"
+        rpy="0 0 0" />
+      <geometry>
+        <mesh
+          filename="package://vega_description/meshes/Link_5.STL"
+          scale="0.001 0.001 0.001" />
       </geometry>
     </collision>
@@ -435,19 +437,21 @@
       <geometry>
         <mesh
-          filename="package://vega_description/meshes/Link_8.STL" />
-      </geometry>
-      <material
-        name="">
-        <color
-          rgba="0.752941176470588 0.752941176470588 0.752941176470588 1" />
-      </material>
-    </visual>
-    <collision>
-      <origin
-        xyz="0 0 0"
-        rpy="0 0 0" />
-      <geometry>
-        <mesh
-          filename="package://vega_description/meshes/Link_8.STL" />
+          filename="package://vega_description/meshes/Link_8.STL"
+          scale="0.001 0.001 0.001" />
+      </geometry>
+      <material
+        name="">
+        <color
+          rgba="0.752941176470588 0.752941176470588 0.752941176470588 1" />
+      </material>
+    </visual>
+    <collision>
+      <origin
+        xyz="0 0 0"
+        rpy="0 0 0" />
+      <geometry>
+        <mesh
+          filename="package://vega_description/meshes/Link_8.STL"
+          scale="0.001 0.001 0.001" />
       </geometry>
     </collision>
@@ -596,5 +600,5 @@
     type="fixed">
     <origin
-      xyz="0.030 -0.020 0"
+      xyz="0.060 -0.054 0.025"
       rpy="0 0 0" />
     <parent
@@ -621,4 +625,25 @@
         izz="0.000541662726314469" />
     </inertial>
+    <visual>
+      <origin
+        xyz="0 -0.01 0"
+        rpy="1.5701 0 0" />
+      <geometry>
+        <cylinder radius="0.0275" length="0.02"/>
+      </geometry>
+      <material
+        name="">
+        <color
+          rgba="0.752941176470588 0.752941176470588 0.752941176470588 1" />
+      </material>
+    </visual>
+    <collision>
+      <origin
+        xyz="0 -0.01 0"
+        rpy="1.5701 0 0" />
+      <geometry>
+        <cylinder radius="0.0275" length="0.02"/>
+      </geometry>
+    </collision>
   </link>
   <joint
@@ -626,5 +651,5 @@
     type="revolute">
     <origin
-      xyz="0.030 0 0"
+      xyz="0 0 0"
       rpy="0 0 0" />
     <parent

Commit message: fixed naming

File: vega_description/urdf/vega_description.xacro (robot description, xacro)
@@ -4,5 +4,5 @@
   name="vega_description">
   <link
-    name="Link_1">
+    name="link_1">
     <inertial>
       <origin
@@ -25,5 +25,5 @@
       <geometry>
         <mesh
-          filename="package://vega_description/meshes/Link_1.STL"/>
+          filename="package://vega_description/meshes/link_1.STL"/>
       </geometry>
       <material
@@ -39,10 +39,10 @@
       <geometry>
         <mesh
-          filename="package://vega_description/meshes/Link_1.STL" />
-      </geometry>
-    </collision>
-  </link>
-  <link
-    name="Link_2">
+          filename="package://vega_description/meshes/link_1.STL" />
+      </geometry>
+    </collision>
+  </link>
+  <link
+    name="link_2">
     <inertial>
       <origin
@@ -65,24 +65,24 @@
       <geometry>
         <mesh
-          filename="package://vega_description/meshes/Link_2.STL" />
-      </geometry>
-      <material
-        name="">
-        <color
-          rgba="0.752941176470588 0.752941176470588 0.752941176470588 1" />
-      </material>
-    </visual>
-    <collision>
-      <origin
-        xyz="0 0 0"
-        rpy="0 0 0" />
-      <geometry>
-        <mesh
-          filename="package://vega_description/meshes/Link_2.STL" />
-      </geometry>
-    </collision>
-  </link>
-  <joint
-    name="Joint_1_2"
+          filename="package://vega_description/meshes/link_2.STL" />
+      </geometry>
+      <material
+        name="">
+        <color
+          rgba="0.752941176470588 0.752941176470588 0.752941176470588 1" />
+      </material>
+    </visual>
+    <collision>
+      <origin
+        xyz="0 0 0"
+        rpy="0 0 0" />
+      <geometry>
+        <mesh
+          filename="package://vega_description/meshes/link_2.STL" />
+      </geometry>
+    </collision>
+  </link>
+  <joint
+    name="joint_1_2"
     type="revolute">
     <origin
@@ -90,7 +90,7 @@
       rpy="1.5707963267949 0 0" />
     <parent
-      link="Link_1" />
-    <child
-      link="Link_2" />
+      link="link_1" />
+    <child
+      link="link_2" />
     <axis
       xyz="0 1 0" />
@@ -102,5 +102,5 @@
   </joint>
   <link
-    name="Link_3">
+    name="link_3">
     <inertial>
       <origin
@@ -123,24 +123,24 @@
       <geometry>
         <mesh
-          filename="package://vega_description/meshes/Link_3.STL" />
-      </geometry>
-      <material
-        name="">
-        <color
-          rgba="0.752941176470588 0.752941176470588 0.752941176470588 1" />
-      </material>
-    </visual>
-    <collision>
-      <origin
-        xyz="0 0 0"
-        rpy="0 0 0" />
-      <geometry>
-        <mesh
-          filename="package://vega_description/meshes/Link_3.STL" />
-      </geometry>
-    </collision>
-  </link>
-  <joint
-    name="Joint_2_3"
+          filename="package://vega_description/meshes/link_3.STL" />
+      </geometry>
+      <material
+        name="">
+        <color
+          rgba="0.752941176470588 0.752941176470588 0.752941176470588 1" />
+      </material>
+    </visual>
+    <collision>
+      <origin
+        xyz="0 0 0"
+        rpy="0 0 0" />
+      <geometry>
+        <mesh
+          filename="package://vega_description/meshes/link_3.STL" />
+      </geometry>
+    </collision>
+  </link>
+  <joint
+    name="joint_2_3"
     type="revolute">
     <origin
@@ -148,7 +148,7 @@
       rpy="-1.5708 0 1.8326" />
     <parent
-      link="Link_2" />
-    <child
-      link="Link_3" />
+      link="link_2" />
+    <child
+      link="link_3" />
     <axis
       xyz="0 1 0" />
@@ -160,5 +160,5 @@
   </joint>
   <link
-    name="Link_4">
+    name="link_4">
     <inertial>
       <origin
@@ -181,55 +181,55 @@
       <geometry>
         <mesh
-          filename="package://vega_description/meshes/Link_4.STL" />
-      </geometry>
-      <material
-        name="">
-        <color
-          rgba="0.752941176470588 0.752941176470588 0.752941176470588 1" />
-      </material>
-    </visual>
-    <collision>
-      <origin
-        xyz="0 0 0"
-        rpy="0 0 0" />
-      <geometry>
-        <mesh
-          filename="package://vega_description/meshes/Link_4.STL" />
-      </geometry>
-    </collision>
-  </link>
-  <link
-    name="Link_3_4">
-  </link>
-  <joint
-    name="Joint_3_4_1"
-    type="continuous">
-    <mimic joint="Joint_2_3" multiplier="-1" offset="0"/>
+          filename="package://vega_description/meshes/link_4.STL" />
+      </geometry>
+      <material
+        name="">
+        <color
+          rgba="0.752941176470588 0.752941176470588 0.752941176470588 1" />
+      </material>
+    </visual>
+    <collision>
+      <origin
+        xyz="0 0 0"
+        rpy="0 0 0" />
+      <geometry>
+        <mesh
+          filename="package://vega_description/meshes/link_4.STL" />
+      </geometry>
+    </collision>
+  </link>
+  <link
+    name="link_3_4">
+  </link>
+  <joint
+    name="joint_3_4_1"
+    type="continuous">
+    <mimic joint="joint_2_3" multiplier="-1" offset="0"/>
     <origin
       xyz="0.25 0.055 0"
       rpy="0 1.309 3.1416" />
     <parent
-      link="Link_3" />
-    <child
-      link="Link_3_4" />
+      link="link_3" />
+    <child
+      link="link_3_4" />
     <axis
       xyz="0 -1 0" />
   </joint>
   <joint
-    name="Joint_3_4_2"
-    type="continuous">
-    <mimic joint="Joint_2_6" multiplier="-1" offset="0"/>
+    name="joint_3_4_2"
+    type="continuous">
+    <mimic joint="joint_2_6" multiplier="-1" offset="0"/>
     <origin
       xyz="0 0 0"
       rpy="0 0 0" />
     <parent
-      link="Link_3_4" />
-    <child
-      link="Link_4" />
+      link="link_3_4" />
+    <child
+      link="link_4" />
     <axis
       xyz="0 -1 0" />
   </joint>
   <link
-    name="Link_5">
+    name="link_5">
     <inertial>
       <origin
@@ -252,5 +252,5 @@
       <geometry>
         <mesh
-          filename="package://vega_description/meshes/Link_5.STL"
+          filename="package://vega_description/meshes/link_5.STL"
           scale="0.001 0.001 0.001" />
       </geometry>
@@ -267,5 +267,5 @@
       <geometry>
         <mesh
-          filename="package://vega_description/meshes/Link_5.STL"
+          filename="package://vega_description/meshes/link_5.STL"
           scale="0.001 0.001 0.001" />
       </geometry>
@@ -273,19 +273,19 @@
   </link>
   <joint
-    name="Joint_4_5"
-    type="continuous">
-    <mimic joint="Joint_2_6" multiplier="-1" offset="0"/>
+    name="joint_4_5"
+    type="continuous">
+    <mimic joint="joint_2_6" multiplier="-1" offset="0"/>
     <origin
       xyz="0.3 0.025 0"
       rpy="-1.5708 0 0" />
     <parent
-      link="Link_4" />
-    <child
-      link="Link_5" />
+      link="link_4" />
+    <child
+      link="link_5" />
     <axis
       xyz="0 0 1" />
   </joint>
   <link
-    name="Link_6">
+    name="link_6">
     <inertial>
       <origin
@@ -308,24 +308,24 @@
       <geometry>
         <mesh
-          filename="package://vega_description/meshes/Link_6.STL" />
-      </geometry>
-      <material
-        name="">
-        <color
-          rgba="0.752941176470588 0.752941176470588 0.752941176470588 1" />
-      </material>
-    </visual>
-    <collision>
-      <origin
-        xyz="0 0 0"
-        rpy="0 0 0" />
-      <geometry>
-        <mesh
-          filename="package://vega_description/meshes/Link_6.STL" />
-      </geometry>
-    </collision>
-  </link>
-  <joint
-    name="Joint_2_6"
+          filename="package://vega_description/meshes/link_6.STL" />
+      </geometry>
+      <material
+        name="">
+        <color
+          rgba="0.752941176470588 0.752941176470588 0.752941176470588 1" />
+      </material>
+    </visual>
+    <collision>
+      <origin
+        xyz="0 0 0"
+        rpy="0 0 0" />
+      <geometry>
+        <mesh
+          filename="package://vega_description/meshes/link_6.STL" />
+      </geometry>
+    </collision>
+  </link>
+  <joint
+    name="joint_2_6"
     type="revolute">
     <origin
@@ -333,7 +333,7 @@
       rpy="0 0 0.17453" />
     <parent
-      link="Link_2" />
-    <child
-      link="Link_6" />
+      link="link_2" />
+    <child
+      link="link_6" />
     <axis
       xyz="0 0 1" />
@@ -345,5 +345,5 @@
   </joint>
   <link
-    name="Link_7">
+    name="link_7">
     <inertial>
       <origin
@@ -366,55 +366,55 @@
       <geometry>
         <mesh
-          filename="package://vega_description/meshes/Link_7.STL" />
-      </geometry>
-      <material
-        name="">
-        <color
-          rgba="0.752941176470588 0.752941176470588 0.752941176470588 1" />
-      </material>
-    </visual>
-    <collision>
-      <origin
-        xyz="0 0 0"
-        rpy="0 0 0" />
-      <geometry>
-        <mesh
-          filename="package://vega_description/meshes/Link_7.STL" />
-      </geometry>
-    </collision>
-  </link>
-  <link
-    name="Link_6_7">
-  </link>
-  <joint
-    name="Joint_6_7_1"
-    type="continuous">
-    <mimic joint="Joint_2_3" multiplier="-1" offset="0"/>
+          filename="package://vega_description/meshes/link_7.STL" />
+      </geometry>
+      <material
+        name="">
+        <color
+          rgba="0.752941176470588 0.752941176470588 0.752941176470588 1" />
+      </material>
+    </visual>
+    <collision>
+      <origin
+        xyz="0 0 0"
+        rpy="0 0 0" />
+      <geometry>
+        <mesh
+          filename="package://vega_description/meshes/link_7.STL" />
+      </geometry>
+    </collision>
+  </link>
+  <link
+    name="link_6_7">
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