Commit message: add ros2 control and launch file

File: vega_description/urdf/vega_description.xacro (robot description, xacro)
@@ -1,667 +1,668 @@
 <?xml version="1.0" encoding="utf-8"?>
 <robot
-  xmlns:xacro="http://www.ros.org/wiki/xacro"
-  name="vega_description">
-  <link
-    name="link_1">
-    <inertial>
-      <origin
-        xyz="1.22743573927168E-05 -2.12020239797617E-06 0.0417491604335673"
-        rpy="0 0 0" />
-      <mass
-        value="1.46638906209098" />
-      <inertia
-        ixx="0.00311535430398331"
-        ixy="2.09807989848561E-07"
-        ixz="1.66649061073481E-07"
-        iyy="0.0031143541425315"
-        iyz="3.36573233719113E-08"
-        izz="0.00545821841694294" />
-    </inertial>
-    <visual>
-      <origin
-        xyz="0 0 0"
-        rpy="1.571 0 0" />
-      <geometry>
-        <mesh
-          filename="package://vega_description/meshes/link_1.STL"/>
-      </geometry>
-      <material
-        name="">
-        <color
-          rgba="0.752941176470588 0.752941176470588 0.752941176470588 1" />
-      </material>
-    </visual>
-    <collision>
-      <origin
-        xyz="0 0 0"
-        rpy="1.571 0 0" />
-      <geometry>
-        <mesh
-          filename="package://vega_description/meshes/link_1.STL" />
-      </geometry>
-    </collision>
-  </link>
-  <link
-    name="link_2">
-    <inertial>
+  xmlns:xacro="http://www.ros.org/wiki/xacro">
+  <xacro:macro name="vega_description">
+    <link
+      name="link_1">
+      <inertial>
+        <origin
+          xyz="1.22743573927168E-05 -2.12020239797617E-06 0.0417491604335673"
+          rpy="0 0 0" />
+        <mass
+          value="1.46638906209098" />
+        <inertia
+          ixx="0.00311535430398331"
+          ixy="2.09807989848561E-07"
+          ixz="1.66649061073481E-07"
+          iyy="0.0031143541425315"
+          iyz="3.36573233719113E-08"
+          izz="0.00545821841694294" />
+      </inertial>
+      <visual>
+        <origin
+          xyz="0 0 0"
+          rpy="1.571 0 0" />
+        <geometry>
+          <mesh
+            filename="package://vega_description/meshes/link_1.STL"/>
+        </geometry>
+        <material
+          name="">
+          <color
+            rgba="0.752941176470588 0.752941176470588 0.752941176470588 1" />
+        </material>
+      </visual>
+      <collision>
+        <origin
+          xyz="0 0 0"
+          rpy="1.571 0 0" />
+        <geometry>
+          <mesh
+            filename="package://vega_description/meshes/link_1.STL" />
+        </geometry>
+      </collision>
+    </link>
+    <link
+      name="link_2">
+      <inertial>
+        <origin
+          xyz="0 0 0"
+          rpy="0 0 0" />
+        <mass
+          value="2.8648922857987" />
+        <inertia
+          ixx="0.0045488257818998"
+          ixy="-0.000195854703692343"
+          ixz="3.21412134183932E-06"
+          iyy="0.00794747497377555"
+          iyz="5.03872017746305E-06"
+          izz="0.00661354256671326" />
+      </inertial>
+      <visual>
+        <origin
+          xyz="0 0 0"
+          rpy="0 0 0" />
+        <geometry>
+          <mesh
+            filename="package://vega_description/meshes/link_2.STL" />
+        </geometry>
+        <material
+          name="">
+          <color
+            rgba="0.752941176470588 0.752941176470588 0.752941176470588 1" />
+        </material>
+      </visual>
+      <collision>
+        <origin
+          xyz="0 0 0"
+          rpy="0 0 0" />
+        <geometry>
+          <mesh
+            filename="package://vega_description/meshes/link_2.STL" />
+        </geometry>
+      </collision>
+    </link>
+    <joint
+      name="joint_1_2"
+      type="revolute">
+      <origin
+        xyz="0 0 0.102"
+        rpy="1.5707963267949 0 0" />
+      <parent
+        link="link_1" />
+      <child
+        link="link_2" />
+      <axis
+        xyz="0 1 0" />
+      <limit
+        lower="-3.142"
+        upper="3.142"
+        effort="10"
+        velocity="2.094" />
+    </joint>
+    <link
+      name="link_3">
+      <inertial>
+        <origin
+          xyz="0.118778332483488 -0.0107730885379603 5.2341464495953E-13"
+          rpy="0 0 0" />
+        <mass
+          value="0.635661384166151" />
+        <inertia
+          ixx="0.000298348623915365"
+          ixy="6.31060272864874E-06"
+          ixz="-5.08825972892271E-14"
+          iyy="0.00448845816808262"
+          iyz="-2.55937357759991E-17"
+          izz="0.00429172562634377" />
+      </inertial>
+      <visual>
+        <origin
+          xyz="0 0 0"
+          rpy="0 0 0" />
+        <geometry>
+          <mesh
+            filename="package://vega_description/meshes/link_3.STL" />
+        </geometry>
+        <material
+          name="">
+          <color
+            rgba="0.752941176470588 0.752941176470588 0.752941176470588 1" />
+        </material>
+      </visual>
+      <collision>
+        <origin
+          xyz="0 0 0"
+          rpy="0 0 0" />
+        <geometry>
+          <mesh
+            filename="package://vega_description/meshes/link_3.STL" />
+        </geometry>
+      </collision>
+    </link>
+    <joint
+      name="joint_2_3"
+      type="revolute">
+      <origin
+        xyz="0.02 0.085 0.0265"
+        rpy="-1.5708 0 1.8326" />
+      <parent
+        link="link_2" />
+      <child
+        link="link_3" />
+      <axis
+        xyz="0 1 0" />
+      <limit
+        lower="-3.142"
+        upper="3.142"
+        effort="50"
+        velocity="2.094" />
+    </joint>
+    <link
+      name="link_4">
+      <inertial>
+        <origin
+          xyz="0.0853087481110666 -0.0109027881973163 0.00273987445096585"
+          rpy="0 0 0" />
+        <mass
+          value="0.445733094117697" />
+        <inertia
+          ixx="0.000124545025927191"
+          ixy="-9.18984884658101E-07"
+          ixz="0.000203813066958736"
+          iyy="0.00609354602814492"
+          iyz="-2.19558292990133E-07"
+          izz="0.00599654478371796" />
+      </inertial>
+      <visual>
+        <origin
+          xyz="0 0 0"
+          rpy="0 0 0" />
+        <geometry>
+          <mesh
+            filename="package://vega_description/meshes/link_4.STL" />
+        </geometry>
+        <material
+          name="">
+          <color
+            rgba="0.752941176470588 0.752941176470588 0.752941176470588 1" />
+        </material>
+      </visual>
+      <collision>
+        <origin
+          xyz="0 0 0"
+          rpy="0 0 0" />
+        <geometry>
+          <mesh
+            filename="package://vega_description/meshes/link_4.STL" />
+        </geometry>
+      </collision>
+    </link>
+    <link
+      name="link_3_4">
+    </link>
+    <joint
+      name="joint_3_4_1"
+      type="continuous">
+      <mimic joint="joint_2_3" multiplier="-1" offset="0"/>
+      <origin
+        xyz="0.25 0.055 0"
+        rpy="0 1.309 3.1416" />
+      <parent
+        link="link_3" />
+      <child
+        link="link_3_4" />
+      <axis
+        xyz="0 -1 0" />
+    </joint>
+    <joint
+      name="joint_3_4_2"
+      type="continuous">
+      <mimic joint="joint_2_6" multiplier="-1" offset="0"/>
       <origin
         xyz="0 0 0"
         rpy="0 0 0" />
-      <mass
-        value="2.8648922857987" />
-      <inertia
-        ixx="0.0045488257818998"
-        ixy="-0.000195854703692343"
-        ixz="3.21412134183932E-06"
-        iyy="0.00794747497377555"
-        iyz="5.03872017746305E-06"
-        izz="0.00661354256671326" />
-    </inertial>
-    <visual>
+      <parent
+        link="link_3_4" />
+      <child
+        link="link_4" />
+      <axis
+        xyz="0 -1 0" />
+    </joint>
+    <link
+      name="link_5">
+      <inertial>
+        <origin
+          xyz="0.00952764383358035 0.00817180619347385 0.0246303315536559"
+          rpy="0 0 0" />
+        <mass
+          value="0.116143592433757" />
+        <inertia
+          ixx="5.42685200550782E-05"
+          ixy="-5.2844222655857E-06"
+          ixz="-1.11803694401409E-06"
+          iyy="4.1289544024263E-05"
+          iyz="-1.03212198470323E-06"
+          izz="5.14314290266057E-05" />
+      </inertial>
+      <visual>
+        <origin
+          xyz="0 0 0"
+          rpy="0 0 0" />
+        <geometry>
+          <mesh
+            filename="package://vega_description/meshes/link_5.STL"
+            scale="0.001 0.001 0.001" />
+        </geometry>
+        <material
+          name="">
+          <color
+            rgba="0.752941176470588 0.752941176470588 0.752941176470588 1" />
+        </material>
+      </visual>
+      <collision>
+        <origin
+          xyz="0 0 0"
+          rpy="0 0 0" />
+        <geometry>
+          <mesh
+            filename="package://vega_description/meshes/link_5.STL"
+            scale="0.001 0.001 0.001" />
+        </geometry>
+      </collision>
+    </link>
+    <joint
+      name="joint_4_5"
+      type="continuous">
+      <mimic joint="joint_2_6" multiplier="-1" offset="0"/>
+      <origin
+        xyz="0.3 0.025 0"
+        rpy="-1.5708 0 0" />
+      <parent
+        link="link_4" />
+      <child
+        link="link_5" />
+      <axis
+        xyz="0 0 1" />
+    </joint>
+    <link
+      name="link_6">
+      <inertial>
+        <origin
+          xyz="-0.0497529093598293 -1.11022302462516E-16 -0.00976909265143127"
+          rpy="0 0 0" />
+        <mass
+          value="0.140467568500251" />
+        <inertia
+          ixx="3.35801010666134E-05"
+          ixy="-8.86063009396581E-20"
+          ixz="-9.81693731169107E-07"
+          iyy="0.000250818338085388"
+          iyz="-7.81409448092477E-22"
+          izz="0.00027533816649807" />
+      </inertial>
+      <visual>
+        <origin
+          xyz="0 0 0"
+          rpy="0 0 0" />
+        <geometry>
+          <mesh
+            filename="package://vega_description/meshes/link_6.STL" />
+        </geometry>
+        <material
+          name="">
+          <color
+            rgba="0.752941176470588 0.752941176470588 0.752941176470588 1" />
+        </material>
+      </visual>
+      <collision>
+        <origin
+          xyz="0 0 0"
+          rpy="0 0 0" />
+        <geometry>
+          <mesh
+            filename="package://vega_description/meshes/link_6.STL" />
+        </geometry>
+      </collision>
+    </link>
+    <joint
+      name="joint_2_6"
+      type="revolute">
+      <origin
+        xyz="0.02 0.085 -0.0285"
+        rpy="0 0 0.17453" />
+      <parent
+        link="link_2" />
+      <child
+        link="link_6" />
+      <axis
+        xyz="0 0 1" />
+      <limit
+        lower="-3.142"
+        upper="3.142"
+        effort="15"
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